File: design/MeshRepeater2_Logic/MeshRepeater2_Logic.kicad_sch (KiCad schematic)
At the start: 22 parts, among them J13 SMA 50Ohm, M1 NiceNano_CLONE_MODIFIED, M2 HT-RA62, SW1 USER, SW2 RESET

Commit message: Publish Mesh Repeater 2.0 A3 prototype and engineering audit
Connections:
- net RADIO_3V3: now also FB1.1; no longer C23.1, C24.1, FB1.2, M2.3 (3V3)
- net SYS_3V3: no longer FB1.1
- new net RADIO_LOCAL_3V3: C23.1, C24.1, FB1.2, M2.3 (3V3)
Other:
- note added: "3V3 через J11 на POWER; RAW/BAT: NC. USB-зарядник отключить. Снять шунт J11 ДО подключения USB. Вернуть J11 только после отключения USB."
- note added: "POWER: J11 → NT2-звезда → две ветви. Модем: RADIO_3V3 → FB1 → RADIO_LOCAL_3V3."
- note added: "V2.0-A3 / 2026-10-13 / инженерный прототип"
- note removed: "3V3 через J11; RAW/BAT: NC. USB-зарядник отключить. Снять шунт J11 ДО подключения USB. Вернуть J11 только после отключения USB."
- note removed: "V2.0-A2 / 2026-10-12 / инженерный прототип"
- note removed: "Модем: отдельная ветвь J11 → FB1 → RADIO_3V3. GPS/RTC питаются до FB1."
