File: design/MeshRepeater2_Logic/RTC_IO.kicad_sch (KiCad schematic)
At the start: 18 parts, among them J3 I2C3V3, J4 GPS / T114 P3, J5 UART3V3, Q2 AO3401A, Q3 2N7002K, U4 DS3231MZ+TRL, U7 SN74LVC2G125

Commit message: Publish Mesh Repeater 2.0 A3 prototype and engineering audit
Other:
- note added: "V2.0-A3 / 2026-10-13 / инженерный прототип"
- note removed: "V2.0-A2 / 2026-10-12 / инженерный прототип"
