File: design/MeshRepeater2_Logic/Watchdog.kicad_sch (KiCad schematic)
At the start: 8 parts, among them J10 AVR ISP 3V3, U6 ATtiny13A-SSU

Commit message: Publish Mesh Repeater 2.0 A3 prototype and engineering audit
Other:
- note added: "V2.0-A3 / 2026-10-13 / инженерный прототип"
- note removed: "V2.0-A2 / 2026-10-12 / инженерный прототип"
