File: design/MeshRepeater2_Power/BatteryMonitor.kicad_sch (KiCad schematic)
At the start: 7 parts, among them J8 Na-ion 1S, U12 INA219AIDR

Commit message: Publish Mesh Repeater 2.0 A3 prototype and engineering audit
Parts:
- J8: value Na-ion 1S -> Na-ion; Value_LTO_2S Na-ion 1S -> Na-ion; Value_NaIon Na-ion 1S -> Na-ion; Value_NaIon_NoCold Na-ion 1S -> Na-ion
- R71: footprint Meshcore:R_2512_6332Metric__V2_R71 -> Meshcore:R_2512_6332Metric__A3_R71
Other:
- note added: "2512 / 6.3 x 3.2 mm"
- note added: "V2.0-A3 / 2026-10-13 / инженерный прототип"
- note added: "Питание VS: SYS_3V3 после J11 на POWER; USB через J101.1/3 при снятой J11."
- note removed: "2512 / 1W"
- note removed: "V2.0-A2 / 2026-10-12 / инженерный прототип"
- note removed: "Питание VS: SYS_3V3 с LOGIC через J101.7; работает при USB и снятой J11."
