File: design/MeshRepeater2_Power/Converter.kicad_sch (KiCad schematic)
At the start: 43 parts, among them U2 TPS63802DLAR

Commit message: Publish Mesh Repeater 2.0 A3 prototype and engineering audit
Parts:
- R40: footprint Meshcore:R_Vishay_WSL1206_18__V2_R40 -> Meshcore:R_Vishay_WSL2512_A3__A3_R40; MPN WSL1206R0220FEA -> WSL2512R0220FEA; MPN_LTO_2S WSL1206R0220FEA -> WSL2512R0220FEA; MPN_NaIon WSL1206R0220FEA -> WSL2512R0220FEA; MPN_NaIon_NoCold WSL1206R0220FEA -> WSL2512R0220FEA
- R41: footprint Meshcore:R_Vishay_WSL1206_18__V2_R41 -> Meshcore:R_Vishay_WSL2512_A3__A3_R41; MPN WSL1206R0220FEA -> WSL2512R0220FEA; MPN_LTO_2S WSL1206R0220FEA -> WSL2512R0220FEA; MPN_NaIon WSL1206R0220FEA -> WSL2512R0220FEA; MPN_NaIon_NoCold WSL1206R0220FEA -> WSL2512R0220FEA
- R55: footprint Meshcore:R_Vishay_WSL1206_18__V2_R55 -> Meshcore:R_Vishay_WSL2512_A3__A3_R55; MPN WSL1206R0470FEA -> WSL2512R0470FEA; MPN_LTO_2S WSL1206R0470FEA -> WSL2512R0470FEA; MPN_NaIon WSL1206R0470FEA -> WSL2512R0470FEA; MPN_NaIon_NoCold WSL1206R0470FEA -> WSL2512R0470FEA; Vendor URL https://www.chipdip.ru/product/wsl1206r0470fea-current-sens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 -> (none)
- TP1: footprint Meshcore:TestPoint_Pad_D1.5mm__V2_TP1 -> Meshcore:TestPoint_Pad_D1p5mm_A3_Edge_R0p9
- TP6: footprint Meshcore:TestPoint_Pad_D1.5mm__V2_TP6 -> Meshcore:TestPoint_Pad_D1p5mm_A3_Edge_R0p9
Other:
- note added: "2512 / 6.3 x 3.2 mm"
- note added: "FILTER_OUT → J11 → NT2-звезда на листе Interconnect (POWER)."
- note added: "V2.0-A3 / 2026-10-13 / инженерный прототип"
- note added: "WSL2512R0220FEA"
- note added: "WSL2512R0470FEA"
- note removed: "1206 / 0.25 W"
- note removed: "FILTER_OUT → межплатные штыри → J11.1 (LOGIC)."
- note removed: "R0470FEA"
- note removed: "V2.0-A2 / 2026-10-12 / инженерный прототип"
- note removed: "WSL1206"
- note removed: "WSL1206, 1206 (3216)"
- note removed: "WSL1206R0220FEA"
