File: design/MeshRepeater2_Power/Interconnect.kicad_sch (KiCad schematic)
At the start: 5 parts, among them J101 INTERBOARD 2x6 VERTICAL

Commit message: Publish Mesh Repeater 2.0 A3 prototype and engineering audit
Parts:
- added J11: LC OUT - 3V3, Meshcore:Connfly_DS1022_1x02RUF11_B_Horizontal, symbol Meshcore:JUMPER_H
- added NT2: 3V3 STAR, Meshcore:NetTie_2_SMD_Power_Star_A3, symbol Meshcore:NETTIE
Connections:
- net FILTER_OUT: now also J11.1; no longer J101.1 (FILTER_OUT), J101.3 (FILTER_OUT), J101.5 (FILTER_OUT)
- net GND: no longer J101.8 (GND)
- net SYS_3V3: now also J101.1 (SYS_3V3), J101.3 (SYS_3V3), J11.2, NT2.1; no longer J101.7 (SYS_3V3)
- new net RADIO_3V3: J101.5 (RADIO_3V3), J101.7 (RADIO_3V3), NT2.2
- no-connect marks 0 -> 1
Other:
- note added: "1x2 / 2.54 / 90deg"
- note added: "BAT: отвод измерения прямо от разъёма батареи, до R71."
- note added: "DS1022-1x40RUF11-B"
- note added: "INA219 питается от SYS_3V3; при снятой J11 его питает USB через штыри."
- note added: "NT2 — медная звезда, не устанавливаемая деталь. Не разрезать."
- note added: "SYS_3V3 → NiceNano и периферия; RADIO_3V3 → только модем через FB1."
- note added: "V2.0-A3 / 2026-10-13 / инженерный прототип"
- note added: "Один шунт J11: снять ДО USB; вернуть после отключения USB."
- note removed: "BAT: отдельный отвод измерения прямо от разъёма батареи."
- note removed: "SYS_3V3 возвращается с LOGIC только для питания INA219."
- note removed: "V2.0-A2 / 2026-10-12 / инженерный прототип"
- note removed: "Основные токи FILTER_OUT и GND идут через вертикальные штыри."
