File: design/MeshRepeater2_Power/LTO_Balancer.kicad_sch (KiCad schematic)
At the start: 13 parts, among them J12 LTO 2S + MID -, U8 LMV431A, U9 LMV431A

Commit message: Publish Mesh Repeater 2.0 A3 prototype and engineering audit
Parts:
- J12: value LTO 2S + MID - -> LTO; Value_LTO_2S LTO 2S + MID - -> LTO; Value_NaIon LTO 2S + MID - -> LTO; Value_NaIon_NoCold LTO 2S + MID - -> LTO
Other:
- note added: "V2.0-A3 / 2026-10-13 / инженерный прототип"
- note added: "V2.0-A3: отдельной защиты ячеек и защиты от перенапряжения нет."
- note removed: "V2.0-A2 / 2026-10-12 / инженерный прототип"
- note removed: "V2.0-A2: отдельной защиты ячеек и защиты от перенапряжения нет."
