File: design/MeshRepeater2_Power/MeshRepeater2_Power.kicad_sch (KiCad schematic)
At the start: 29 parts, among them J7 SOLAR 12V, Q1 AO3401A, U1 CN3722

Commit message: Publish Mesh Repeater 2.0 A3 prototype and engineering audit
Parts:
- R1: footprint Meshcore:R_1206_3216Metric__V2_R1 -> Meshcore:R_Vishay_WSL2512_A3__A3_R1; MPN PT1206FR-7W0R28L -> WSL2512R2800FEA; MPN_LTO_2S PT1206FR-7W0R28L -> WSL2512R2800FEA; MPN_NaIon PT1206FR-7W0R28L -> WSL2512R2800FEA; MPN_NaIon_NoCold PT1206FR-7W0R28L -> WSL2512R2800FEA
- R56: value 1.8 ohm 1% 0.125W -> 1.8R 1% 1W; footprint Meshcore:R_0805_2012Metric__V2_R56 -> Meshcore:R_2512_6332Metric__A3_R56; MPN RC0805FR-071R8L -> RC2512FK-071R8L; MPN_LTO_2S RC0805JR-070RL -> RC2512JK-070RL; MPN_NaIon RC0805FR-071R8L -> RC2512FK-071R8L; MPN_NaIon_NoCold RC0805JR-070RL -> RC2512JK-070RL; Value_NaIon 1.8 ohm 1% 0.125W -> 1.8R 1% 1W; Vendor URL https://www.danomsk.ru/shop/6-rezistory/86-rezistory-postoy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 -> (none)
- TP9: footprint Meshcore:TestPoint_Pad_D1.5mm__V2_TP9 -> Meshcore:TestPoint_Pad_D1p5mm_A3_Edge_R0p9
Other:
- note added: "2512 / 6.3 x 3.2 mm"
- note added: "RC2512FK-071R8L"
- note added: "V2.0-A3 / 2026-10-13 / инженерный прототип"
- note added: "WSL2512R2800FEA"
- note removed: "7W0R28L"
- note removed: "PT1206FR-"
- note removed: "RC0805FR-071R8L"
- note removed: "V2.0-A2 / 2026-10-12 / инженерный прототип"
