File: design/MeshRepeater2_Power/Thermal.kicad_sch (KiCad schematic)
At the start: 24 parts, among them Q4 AO3401A, Q5 BSS138, Q6 AO3401A, Q7 AO3401A, U10 LM393XK, U11 LM285Z-2.5G

Commit message: Publish Mesh Repeater 2.0 A3 prototype and engineering audit
Other:
- note added: "V2.0-A3 / 2026-10-13 / инженерный прототип"
- note removed: "V2.0-A2 / 2026-10-12 / инженерный прототип"
